File: PCB/Timer_Counter/Timer_Counter.kicad_sch (KiCad schematic)
At the start: 7 parts, among them J1 Conn_01x20, J2 Conn_01x20, J3 Conn_01x06, J4 Conn_01x03, J5 Conn_01x05

Commit message: Them pcb mơi sửa vào
Parts:
- DS3231: renamed from J3; footprint (none) -> Connector_PinSocket_2.54mm:PinSocket_1x06_P2.54mm_Vertical
- IR1: renamed from J4; footprint Connector_PinHeader_2.54mm:PinHeader_1x03_P2.54mm_Vertical -> Connector_PinSocket_2.54mm:PinSocket_1x03_P2.54mm_Vertical
- J1, J2: footprint Connector_PinHeader_2.54mm:PinHeader_1x20_P2.54mm_Vertical -> Connector_PinSocket_2.54mm:PinSocket_1x20_P2.54mm_Vertical
- LD2410c1: renamed from J5; footprint (none) -> Connector_PinSocket_2.54mm:PinSocket_1x05_P2.54mm_Horizontal
- Oled1: footprint Connector_PinHeader_2.54mm:PinHeader_1x04_P2.54mm_Vertical -> Connector_PinSocket_2.54mm:PinSocket_1x04_P2.54mm_Horizontal
Connections:
- net G is gone; now on net GND: IR1.1 (Pin_1), Oled1.1 (Pin_1)
- net +3.3V: now also Oled1.2 (Pin_2); no longer J2.3 (Pin_3)
- net +5V: now also DS3231.2 (Pin_2), IR1.2 (Pin_2), LD2410c1.1 (Pin_1)
- net OUT: now also J1.5 (Pin_5)
- net SCL: now also Oled1.3 (Pin_3)
- net SDA: now also Oled1.4 (Pin_4)
- removed net 5V: DS3231.2 (Pin_2), IR1.2 (Pin_2), LD2410c1.1 (Pin_1), Oled1.2 (Pin_2)
- net SCL2: no longer names the net of J2.6 (Pin_6)
- net SCL2: no longer Oled1.3 (Pin_3)
- net SDA2: no longer names the net of J2.5 (Pin_5)
- net SDA2: no longer Oled1.4 (Pin_4)
Changed lines of the file:
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@@
-	)
-	(junction
-		(at 125.73 115.57)
-		(diameter 0)
-		(color 0 0 0 0)
-	)
-	(junction
-		(at 182.88 72.39)
-		(diameter 0)
-		(color 0 0 0 0)
 	)
 	(junction
@@
 	)
 	(no_connect
+		(at 170.18 77.47)
+	)
+	(no_connect
 		(at 144.78 97.79)
 	)
@@
 	)
 	(no_connect
-		(at 62.23 74.93)
-	)
-	(no_connect
 		(at 170.18 69.85)
 	)
@@
 	)
 	(no_connect
-		(at 62.23 72.39)
-	)
-	(no_connect
 		(at 170.18 74.93)
 	)
@@
 	)
 	(no_connect
-		(at 144.78 77.47)
-	)
-	(no_connect
 		(at 144.78 95.25)
 	)
 	(no_connect
+		(at 170.18 80.01)
+	)
+	(no_connect
 		(at 144.78 87.63)
 	)
@@
 	)
 	(no_connect
+		(at 170.18 72.39)
+	)
+	(no_connect
 		(at 144.78 90.17)
 	)
@@
 	(wire
 		(pts
-			(xy 170.18 72.39) (xy 182.88 72.39)
-		)
-		(stroke
-			(width 0)
-			(type default)
-		)
-	)
-	(wire
-		(pts
 			(xy 140.97 72.39) (xy 144.78 72.39)
 		)
@@
 	(wire
 		(pts
-			(xy 170.18 77.47) (xy 172.72 77.47)
-		)
-		(stroke
-			(width 0)
-			(type default)
-		)
-	)
-	(wire
-		(pts
 			(xy 140.97 82.55) (xy 144.78 82.55)
 		)
@@
 	(wire
 		(pts
+			(xy 60.96 72.39) (xy 62.23 72.39)
+		)
+		(stroke
+			(width 0)
+			(type default)
+		)
+	)
+	(wire
+		(pts
 			(xy 102.87 129.54) (xy 102.87 125.73)
 		)
@@
 	(wire
 		(pts
-			(xy 118.11 115.57) (xy 125.73 115.57)
-		)
-		(stroke
-			(width 0)
-			(type default)
-		)
-	)
-	(wire
-		(pts
-			(xy 173.99 80.01) (xy 170.18 80.01)
-		)
-		(stroke
-			(width 0)
-			(type default)
-		)
-	)
-	(wire
-		(pts
 			(xy 125.73 104.14) (xy 125.73 113.03)
 		)
@@
 	(wire
 		(pts
-			(xy 125.73 123.19) (xy 125.73 115.57)
-		)
-		(stroke
-			(width 0)
-			(type default)
-		)
-	)
-	(wire
-		(pts
 			(xy 144.78 67.31) (xy 140.97 67.31)
 		)
@@
 	(wire
 		(pts
-			(xy 125.73 115.57) (xy 144.78 115.57)
+			(xy 118.11 115.57) (xy 144.78 115.57)
 		)
 		(stroke
@@
 	(wire
 		(pts
-			(xy 182.88 123.19) (xy 125.73 123.19)
-		)
-		(stroke
-			(width 0)
-			(type default)
-		)
-	)
-	(wire
-		(pts
 			(xy 107.95 129.54) (xy 107.95 125.73)
 		)
@@
 	(wire
 		(pts
+			(xy 140.97 77.47) (xy 144.78 77.47)
+		)
+		(stroke
+			(width 0)
+			(type default)
+		)
+	)
+	(wire
+		(pts
 			(xy 191.77 92.71) (xy 195.58 92.71)
 		)
@@
 		(pts
 			(xy 140.97 85.09) (xy 144.78 85.09)
-		)
-		(stroke
-			(width 0)
-			(type default)
-		)
-	)
-	(wire
-		(pts
-			(xy 182.88 72.39) (xy 182.88 123.19)
 		)
 		(stroke
@@
 		)
 	)
-	(label "SDA2"
-		(at 172.72 77.47 0)
-		(effects
-			(font
-				(size 1.27 1.27)
-			)
-			(justify left bottom)
-		)
-	)
-	(label "5V"
+	(label "+5V"
 		(at 62.23 64.77 180)
 		(effects
@@
 		)
 	)
-	(label "5V"
+	(label "+3.3V"
 		(at 109.22 74.93 270)
-		(effects
-			(font
-				(size 1.27 1.27)
-			)
-			(justify right bottom)
-		)
-	)
-	(label "SCL2"
-		(at 173.99 80.01 180)
 		(effects
 			(font
@@
 	)
 	(label "RX"
-		(at 62.23 72.39 180)
+		(at 60.96 72.39 180)
 		(effects
 			(font
@@
 		)
 	)
-	(label "SDA2"
+	(label "SDA"
 		(at 114.3 74.93 270)
 		(effects
@@
 		)
 	)
-	(label "SCL2"
+	(label "OUT"
+		(at 140.97 77.47 180)
+		(effects
+			(font
+				(size 1.27 1.27)
+			)
+			(justify right bottom)
+		)
+	)
+	(label "SCL"
 		(at 111.76 74.93 270)
 		(effects
@@
 		)
 	)
-	(label "5V"
+	(label "+5V"
 		(at 191.77 90.17 0)
 		(effects
@@
 		)
 	)
-	(label "G"
+	(label "GND"
 		(at 191.77 87.63 0)
 		(effects
@@
 		)
 	)
-	(label "G"
+	(label "GND"
 		(at 106.68 74.93 270)
 		(effects
@@
 		)
 	)
-	(label "5V"
+	(label "+5V"
 		(at 81.28 86.36 180)
 		(effects
@@
 			)
 		)
-		(property "Footprint" "Connector_PinHeader_2.54mm:PinHeader_1x20_P2.54mm_Vertical"
+		(property "Footprint" "Connector_PinSocket_2.54mm:PinSocket_1x20_P2.54mm_Vertical"
 			(at 165.1 90.17 0)
 			(hide yes)
@@
 			)
 		)
-		(property "Footprint" "Connector_PinHeader_2.54mm:PinHeader_1x04_P2.54mm_Vertical"
+		(property "Footprint" "Connector_PinSocket_2.54mm:PinSocket_1x04_P2.54mm_Horizontal"
 			(at 109.22 66.04 0)
 			(hide yes)
@@
 				(path "/9a878fa1-ed82-4704-a9ec-44c13080c227"
 					(reference "Oled1")
-					(unit 1)
-				)
-			)
-		)
-	)
-	(symbol
-		(lib_id "power:PWR_FLAG")
-		(at 182.88 72.39 0)
-		(unit 1)
-		(body_style 1)
-		(exclude_from_sim no)
-		(in_bom yes)
-		(on_board yes)
-		(in_pos_files yes)
-		(dnp no)
-		(fields_autoplaced yes)
-		(property "Reference" "#FLG01"
-			(at 182.88 70.485 0)
-			(hide yes)
-			(show_name no)
-			(do_not_autoplace no)
-			(effects
-				(font
-					(size 1.27 1.27)
-				)
-			)
-		)
-		(property "Value" "PWR_FLAG"
-			(at 182.88 67.31 0)
-			(show_name no)
-			(do_not_autoplace no)
-			(effects
-				(font
-					(size 1.27 1.27)
-				)
-			)
-		)
-		(property "Footprint" ""
-			(at 182.88 72.39 0)
-			(hide yes)
-			(show_name no)
-			(do_not_autoplace no)
-			(effects
-				(font
-					(size 1.27 1.27)
-				)
-			)
-		)
-		(property "Datasheet" ""
-			(at 182.88 72.39 0)
-			(hide yes)
-			(show_name no)
-			(do_not_autoplace no)
-			(effects
-				(font
-					(size 1.27 1.27)
-				)
-			)
-		)
-		(property "Description" "Special symbol for telling ERC where power comes from"
-			(at 182.88 72.39 0)
-			(hide yes)
-			(show_name no)
-			(do_not_autoplace no)
-			(effects
-				(font
-					(size 1.27 1.27)
-				)
-			)
-		)
-		(pin "1"
-		)
-		(instances
-			(project "Timer_Counter"
-				(path "/9a878fa1-ed82-4704-a9ec-44c13080c227"
-					(reference "#FLG01")
 					(unit 1)
 				)
@@
 			)
 		)
-		(property "Footprint" "Connector_PinHeader_2.54mm:PinHeader_1x20_P2.54mm_Vertical"
+		(property "Footprint" "Connector_PinSocket_2.54mm:PinSocket_1x20_P2.54mm_Vertical"
 			(at 149.86 90.17 0)
 			(hide yes)
@@
 		(dnp no)
 		(fields_autoplaced yes)
-		(property "Reference" "J5"
+		(property "Reference" "LD2410c1"
 			(at 69.85 68.5799 0)
 			(show_name no)
@@
 			)
 		)
-		(property "Footprint" ""
+		(property "Footprint" "Connector_PinSocket_2.54mm:PinSocket_1x05_P2.54mm_Horizontal"
 			(at 67.31 69.85 0)
 			(hide yes)
@@
 			(project "Timer_Counter"
 				(path "/9a878fa1-ed82-4704-a9ec-44c13080c227"
-					(reference "J5")
+					(reference "LD2410c1")
 					(unit 1)
 				)
@@
 		(dnp no)
 		(fields_autoplaced yes)
-		(property "Reference" "J3"
+		(property "Reference" "DS3231"
 			(at 88.9 88.8999 0)
 			(show_name no)
@@
 			)
 		)
-		(property "Footprint" ""
+		(property "Footprint" "Connector_PinSocket_2.54mm:PinSocket_1x06_P2.54mm_Vertical"
 			(at 86.36 88.9 0)
 			(hide yes)
@@
 			(project "Timer_Counter"
 				(path "/9a878fa1-ed82-4704-a9ec-44c13080c227"
-					(reference "J3")
+					(reference "DS3231")
 					(unit 1)
 				)
@@
 		(dnp no)
 		(fields_autoplaced yes)
-		(property "Reference" "J4"
+		(property "Reference" "IR1"
 			(at 203.2 88.8999 0)
 			(show_name no)
@@
 			)
 		)
-		(property "Footprint" "Connector_PinHeader_2.54mm:PinHeader_1x03_P2.54mm_Vertical"
+		(property "Footprint" "Connector_PinSocket_2.54mm:PinSocket_1x03_P2.54mm_Vertical"
 			(at 200.66 90.17 0)
 			(hide yes)
@@
 			(project "Timer_Counter"
 				(path "/9a878fa1-ed82-4704-a9ec-44c13080c227"
-					(reference "J4")
+					(reference "IR1")
 					(unit 1)
 				)

Commit message: Cập nhật file PCB
Parts:
- added ESP01: Conn_02x04_Odd_Even, Connector_PinSocket_2.54mm:PinSocket_2x04_P2.54mm_Vertical, symbol Connector_Generic:Conn_02x04_Odd_Even
Connections:
- net +3.3V: now also ESP01.1 (Pin_1)
- net A11: now also Key_pad1.5 (Pin_5); no longer Key_pad1.6 (Pin_6)
- net GND: now also J2.1 (Pin_1), ESP01.8 (Pin_8)
- net RX: now also J2.14 (Pin_14)
- net TX: now also J2.13 (Pin_13)
- net En: now reaches J2.6 (Pin_6)
- net En: now also ESP01.5 (Pin_5)
- net RX1: now reaches J1.6 (Pin_6)
- net RX1: now also ESP01.2 (Pin_2)
- net A12: now reaches J1.9 (Pin_9)
- net A12: now also Key_pad1.6 (Pin_6)
- net A10 renamed TX1
- net TX1: now also ESP01.7 (Pin_7); no longer Key_pad1.5 (Pin_5)
- net OUT: no longer names the net of J1.5 (Pin_5)
- net OUT: no longer LD2410c1.3 (Pin_3)
- new net GPIO0: ESP01.4 (Pin_4)
- new net GPIO2: ESP01.6 (Pin_6)
- new net RST: ESP01.3 (Pin_3)
- no-connect marks 27 -> 23

Commit message: Cap nhat file thiet ke PCB
Parts:
- added J3: LED, Connector_PinSocket_2.00mm:PinSocket_1x02_P2.00mm_Vertical, symbol Connector_Generic:Conn_01x02
Connections:
- net GND: now also J3.2 (Pin_2)
- net A0: now reaches J2.16 (Pin_16)
- net A0: now also J3.1 (Pin_1)
- no-connect marks 23 -> 22
Changed lines of the file:
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@@
-	)
-	(no_connect
-		(at 170.18 105.41)
 	)
 	(no_connect
@@
 	(wire
 		(pts
+			(xy 175.26 105.41) (xy 170.18 105.41)
+		)
+		(stroke
+			(width 0)
+			(type default)
+		)
+	)
+	(wire
+		(pts
 			(xy 140.97 72.39) (xy 144.78 72.39)
 		)
@@
 		)
 	)
+	(label "A0"
+		(at 67.31 46.99 180)
+		(effects
+			(font
+				(size 1.27 1.27)
+			)
+			(justify right bottom)
+		)
+	)
 	(label "SQW"
 		(at 81.28 93.98 180)
@@
 		)
 	)
+	(label "GND"
+		(at 67.31 49.53 180)
+		(effects
+			(font
+				(size 1.27 1.27)
+			)
+			(justify right bottom)
+		)
+	)
 	(label "SCL"
 		(at 111.76 74.93 270)
@@
 			)
 			(justify right bottom)
+		)
+	)
+	(label "A0"
+		(at 175.26 105.41 0)
+		(effects
+			(font
+				(size 1.27 1.27)
+			)
+			(justify left bottom)
 		)
 	)
@@
 					(unit 1)
 				)
+			)
+		)
+	)
+	(symbol
+		(lib_id "Connector_Generic:Conn_01x02")
+		(at 72.39 46.99 0)
+		(unit 1)
+		(body_style 1)
+		(exclude_from_sim no)
+		(in_bom yes)
+		(on_board yes)
+		(in_pos_files yes)
+		(dnp no)
+		(fields_autoplaced yes)
+		(property "Reference" "J3"
+			(at 74.93 46.9899 0)
+			(show_name no)
+			(do_not_autoplace no)
+			(effects
+				(font
+					(size 1.27 1.27)
+				)
+				(justify left)
+			)
+		)
+		(property "Value" "LED"
+			(at 74.93 49.5299 0)
+			(show_name no)
+			(do_not_autoplace no)
+			(effects
+				(font
+					(size 1.27 1.27)
+				)
+				(justify left)
+			)
+		)
+		(property "Footprint" "Connector_PinSocket_2.00mm:PinSocket_1x02_P2.00mm_Vertical"
+			(at 72.39 46.99 0)
+			(hide yes)
+			(show_name no)
+			(do_not_autoplace no)
+			(effects
+				(font
+					(size 1.27 1.27)
+				)
+			)
+		)
+		(property "Datasheet" ""
+			(at 72.39 46.99 0)
+			(hide yes)
+			(show_name no)
+			(do_not_autoplace no)
+			(effects
+				(font
+					(size 1.27 1.27)
+				)
+			)
+		)
+		(property "Description" "Generic connector, single row, 01x02, script generated (kicad-library-utils/schlib/autogen/connector/)"
+			(at 72.39 46.99 0)
+			(hide yes)
+			(show_name no)
+			(do_not_autoplace no)
+			(effects
+				(font
+					(size 1.27 1.27)
+				)
+			)
+		)
+		(pin "1"
+		)
+		(pin "2"
+		)
+		(instances
+			(project "Timer_Counter"
+				(path "/9a878fa1-ed82-4704-a9ec-44c13080c227"
+					(reference "J3")
+					(unit 1)
+				)
